File: schematics/SevSeg.sch (KiCad schematic (older format))
At the start: 17 parts, among them Q1 Q_PNP_BEC, Q2 Q_PNP_BEC, Q3 Q_PNP_BEC, Q4 Q_PNP_BEC

Commit message: Clean up schematic
More readable, some notes on components and decisions, and a proper
linear regulator. 7805 4lyfe.
Changed lines of the file:
@@
 $Descr A4 11693 8268
 encoding utf-8
-Sheet 4 5
+Sheet 3 5
 Title ""
 Date ""
@@
 AR Path="/5A99F3E7/5A984FDC" Ref="AFF3"  Part="1"
 AR Path="/5A99F3F5/5A984FDC" Ref="AFF4"  Part="1"
-F 0 "AFF4" H 5725 4275 50  0000 C CNN
+F 0 "AFF3" H 5725 4275 50  0000 C CNN
 F 1 "CC56-12" H 5725 4175 50  0000 C CNN
 F 2 "Displays_7-Segment:CA56-12SYKWA" H 5225 3525 50  0001 C CNN
@@
 AR Path="/5A99F3E7/5A986B66" Ref="#PWR032"  Part="1"
 AR Path="/5A99F3F5/5A986B66" Ref="#PWR028"  Part="1"
-F 0 "#PWR028" H 3725 4700 50  0001 C CNN
+F 0 "#PWR032" H 3725 4700 50  0001 C CNN
 F 1 "GND" H 3725 4800 50  0000 C CNN
 F 2 "" H 3725 4950 50  0001 C CNN
@@
 AR Path="/5A99F3E7/5A9F5B1C" Ref="R62"  Part="1"
 AR Path="/5A99F3F5/5A9F5B1C" Ref="R78"  Part="1"
-F 0 "R78" V 3355 4750 50  0000 C CNN
+F 0 "R62" V 3355 4750 50  0000 C CNN
 F 1 "1K" V 3275 4750 50  0000 C CNN
 F 2 "Resistors_SMD:R_1206_HandSoldering" V 3205 4750 50  0001 C CNN
@@
 AR Path="/5A99F3E7/5A9F5B9D" Ref="R64"  Part="1"
 AR Path="/5A99F3F5/5A9F5B9D" Ref="R80"  Part="1"
-F 0 "R80" V 4730 4750 50  0000 C CNN
+F 0 "R64" V 4730 4750 50  0000 C CNN
 F 1 "1K" V 4650 4750 50  0000 C CNN
 F 2 "Resistors_SMD:R_1206_HandSoldering" V 4580 4750 50  0001 C CNN
@@
 AR Path="/5A99F3E7/5A9F5BEE" Ref="R74"  Part="1"
 AR Path="/5A99F3F5/5A9F5BEE" Ref="R90"  Part="1"
-F 0 "R90" V 6055 4750 50  0000 C CNN
+F 0 "R74" V 6055 4750 50  0000 C CNN
 F 1 "1K" V 5975 4750 50  0000 C CNN
 F 2 "Resistors_SMD:R_1206_HandSoldering" V 5905 4750 50  0001 C CNN
@@
 AR Path="/5A99F3E7/5A9F5C40" Ref="R76"  Part="1"
 AR Path="/5A99F3F5/5A9F5C40" Ref="R92"  Part="1"
-F 0 "R92" V 7380 4750 50  0000 C CNN
+F 0 "R76" V 7380 4750 50  0000 C CNN
 F 1 "1K" V 7300 4750 50  0000 C CNN
 F 2 "Resistors_SMD:R_1206_HandSoldering" V 7230 4750 50  0001 C CNN
@@
 AR Path="/5A99F3E7/5A9F63AA" Ref="#PWR033"  Part="1"
 AR Path="/5A99F3F5/5A9F63AA" Ref="#PWR029"  Part="1"
-F 0 "#PWR029" H 5100 4700 50  0001 C CNN
+F 0 "#PWR033" H 5100 4700 50  0001 C CNN
 F 1 "GND" H 5100 4800 50  0000 C CNN
 F 2 "" H 5100 4950 50  0001 C CNN
@@
 AR Path="/5A99F3E7/5A9F63F4" Ref="#PWR034"  Part="1"
 AR Path="/5A99F3F5/5A9F63F4" Ref="#PWR030"  Part="1"
-F 0 "#PWR030" H 6425 4700 50  0001 C CNN
+F 0 "#PWR034" H 6425 4700 50  0001 C CNN
 F 1 "GND" H 6425 4800 50  0000 C CNN
 F 2 "" H 6425 4950 50  0001 C CNN
@@
 AR Path="/5A99F3E7/5A9F643E" Ref="#PWR035"  Part="1"
 AR Path="/5A99F3F5/5A9F643E" Ref="#PWR031"  Part="1"
-F 0 "#PWR031" H 7750 4700 50  0001 C CNN
+F 0 "#PWR035" H 7750 4700 50  0001 C CNN
 F 1 "GND" H 7750 4800 50  0000 C CNN
 F 2 "" H 7750 4950 50  0001 C CNN
@@
 AR Path="/5A99F3F5/5A9D031E" Ref="R61"  Part="1"
 AR Path="/5A99F3E7/5A9D031E" Ref="R71"  Part="1"
-F 0 "R61" V 5180 2400 50  0000 C CNN
+F 0 "R71" V 5180 2400 50  0000 C CNN
 F 1 "330" V 5100 2400 50  0000 C CNN
 F 2 "Resistors_SMD:R_1206_HandSoldering" V 5030 2400 50  0001 C CNN
@@
 AR Path="/5A99F3F5/5A9D03F9" Ref="R59"  Part="1"
 AR Path="/5A99F3E7/5A9D03F9" Ref="R70"  Part="1"
-F 0 "R59" V 5180 2225 50  0000 C CNN
+F 0 "R70" V 5180 2225 50  0000 C CNN
 F 1 "330" V 5100 2225 50  0000 C CNN
 F 2 "Resistors_SMD:R_1206_HandSoldering" V 5030 2225 50  0001 C CNN
@@
 AR Path="/5A99F3F5/5A9D042E" Ref="R57"  Part="1"
 AR Path="/5A99F3E7/5A9D042E" Ref="R69"  Part="1"
-F 0 "R57" V 5180 2050 50  0000 C CNN
+F 0 "R69" V 5180 2050 50  0000 C CNN
 F 1 "330" V 5100 2050 50  0000 C CNN
 F 2 "Resistors_SMD:R_1206_HandSoldering" V 5030 2050 50  0001 C CNN
@@
 AR Path="/5A99F3F5/5A9D0462" Ref="R56"  Part="1"
 AR Path="/5A99F3E7/5A9D0462" Ref="R68"  Part="1"
-F 0 "R56" V 5180 1875 50  0000 C CNN
+F 0 "R68" V 5180 1875 50  0000 C CNN
 F 1 "330" V 5100 1875 50  0000 C CNN
 F 2 "Resistors_SMD:R_1206_HandSoldering" V 5030 1875 50  0001 C CNN
@@
 AR Path="/5A99F3F5/5A9D04F9" Ref="R55"  Part="1"
 AR Path="/5A99F3E7/5A9D04F9" Ref="R67"  Part="1"
-F 0 "R55" V 5180 1700 50  0000 C CNN
+F 0 "R67" V 5180 1700 50  0000 C CNN
 F 1 "330" V 5100 1700 50  0000 C CNN
 F 2 "Resistors_SMD:R_1206_HandSoldering" V 5030 1700 50  0001 C CNN
@@
 AR Path="/5A99F3F5/5A9D053A" Ref="R54"  Part="1"
 AR Path="/5A99F3E7/5A9D053A" Ref="R66"  Part="1"
-F 0 "R54" V 5180 1525 50  0000 C CNN
+F 0 "R66" V 5180 1525 50  0000 C CNN
 F 1 "330" V 5100 1525 50  0000 C CNN
 F 2 "Resistors_SMD:R_1206_HandSoldering" V 5030 1525 50  0001 C CNN
@@
 AR Path="/5A99F3F5/5A9D057C" Ref="R53"  Part="1"
 AR Path="/5A99F3E7/5A9D057C" Ref="R65"  Part="1"
-F 0 "R53" V 5180 1350 50  0000 C CNN
+F 0 "R65" V 5180 1350 50  0000 C CNN
 F 1 "330" V 5100 1350 50  0000 C CNN
 F 2 "Resistors_SMD:R_1206_HandSoldering" V 5030 1350 50  0001 C CNN
@@
 AR Path="/5A99F3F5/5A9D05C1" Ref="R52"  Part="1"
 AR Path="/5A99F3E7/5A9D05C1" Ref="R63"  Part="1"
-F 0 "R52" V 5180 1175 50  0000 C CNN
+F 0 "R63" V 5180 1175 50  0000 C CNN
 F 1 "330" V 5100 1175 50  0000 C CNN
 F 2 "Resistors_SMD:R_1206_HandSoldering" V 5030 1175 50  0001 C CNN
@@
 AR Path="/5A99F3F5/5A9E12C4" Ref="Q9"  Part="1"
 AR Path="/5A99F3E7/5A9E12C4" Ref="Q13"  Part="1"
-F 0 "Q9" H 3825 4800 50  0000 L CNN
-F 1 "Q_PNP_BEC" H 3825 4700 50  0000 L CNN
+F 0 "Q13" H 3825 4800 50  0000 L CNN
+F 1 "Q_PNP_BEC" H 3825 4625 50  0000 L CNN
 F 2 "TO_SOT_Packages_SMD:SOT-23_Handsoldering" H 3825 4850 50  0001 C CNN
 F 3 "" H 3625 4750 50  0001 C CNN
@@
 AR Path="/5A99F3F5/5A9E1366" Ref="Q10"  Part="1"
 AR Path="/5A99F3E7/5A9E1366" Ref="Q14"  Part="1"
-F 0 "Q10" H 5200 4800 50  0000 L CNN
-F 1 "Q_PNP_BEC" H 5200 4700 50  0000 L CNN
+F 0 "Q14" H 5200 4800 50  0000 L CNN
+F 1 "Q_PNP_BEC" H 5200 4625 50  0000 L CNN
 F 2 "TO_SOT_Packages_SMD:SOT-23_Handsoldering" H 5200 4850 50  0001 C CNN
 F 3 "" H 5000 4750 50  0001 C CNN
@@
 AR Path="/5A99F3F5/5A9E13AE" Ref="Q11"  Part="1"
 AR Path="/5A99F3E7/5A9E13AE" Ref="Q15"  Part="1"
-F 0 "Q11" H 6525 4800 50  0000 L CNN
-F 1 "Q_PNP_BEC" H 6525 4700 50  0000 L CNN
+F 0 "Q15" H 6525 4800 50  0000 L CNN
+F 1 "Q_PNP_BEC" H 6525 4625 50  0000 L CNN
 F 2 "TO_SOT_Packages_SMD:SOT-23_Handsoldering" H 6525 4850 50  0001 C CNN
 F 3 "" H 6325 4750 50  0001 C CNN
@@
 AR Path="/5A99F3F5/5A9E13FE" Ref="Q12"  Part="1"
 AR Path="/5A99F3E7/5A9E13FE" Ref="Q16"  Part="1"
-F 0 "Q12" H 7850 4800 50  0000 L CNN
-F 1 "Q_PNP_BEC" H 7850 4700 50  0000 L CNN
+F 0 "Q16" H 7850 4800 50  0000 L CNN
+F 1 "Q_PNP_BEC" H 7850 4625 50  0000 L CNN
 F 2 "TO_SOT_Packages_SMD:SOT-23_Handsoldering" H 7850 4850 50  0001 C CNN
 F 3 "" H 7650 4750 50  0001 C CNN
