File: schematics/long_count.kicad_pcb (KiCad board)
At the start: 2 copper layers, 148.6 x 59.7 mm, 122 parts, among them J1 PICKIT connector, J2 BARREL_JACK, Q1 Q_PNP_BEC, Q10 Q_PNP_BEC, Q11 Q_PNP_BEC, Q12 Q_PNP_BEC, Q13 Q_PNP_BEC, Q14 Q_PNP_BEC, Q15 Q_PNP_BEC, Q16 Q_PNP_BEC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

Commit message: remove tracks through pads
Routing:
- net GND: track 67.6 -> 146.7 mm, vias 13 -> 23
- net Net-(C3-Pad2): track 18.2 -> 27.2 mm
- net Net-(F1-Pad2): track 35.2 -> 41.9 mm
- net +5V: track 152.2 -> 155.8 mm
- net ICSPCLK: track 56.9 -> 59.5 mm
- net (no net): track 1.10 -> 0.00 mm, vias 3 -> 0
- net Net-(R24-Pad1): track 65.7 -> 66.3 mm

Commit message: Add test points for VDD and VSS
Also add center positive polarity symbol for DC input
Parts:
- added J3: VDD, Pin_Headers:Pin_Header_Straight_1x01_Pitch2.54mm, F.Cu at (146.3, 70.4)
- added J4: VSS, Pin_Headers:Pin_Header_Straight_1x01_Pitch2.54mm, F.Cu at (98.3, 73.1)
- added REF***: Polarity_Center_Positive_6mm_SilkScreen, Symbols:Polarity_Center_Positive_6mm_SilkScreen, B.Cu at (65.5, 79.5)
Routing:
- net +5V: track 155.8 -> 159.2 mm
